File: label copy.kicad_sch (KiCad schematic)
At the start: 145 parts, among them Q3 BC547, Q4 BC547, Q5 BC547, Q6 BC547, SW11 SW_Push, SW12 SW_Push, SW13 SW_Push, SW14 SW_Push, SW15 SW_Push, SW16 SW_Push, SW17 SW_Push, SW18 SW_Push, SW19 SW_Push, SW20 SW_Push, SW21 SW_Push, SW22 SW_Push, SW23 SW_Push, U1 74HC86, U18 74HCT574, U2 74HC86, U20 74HC86, U21 74HC86, U22 74HC74, U23 74HCT574, U24 74LS194, U25 74LS194, U26 74LS194, U27 74LS194, U28 74LS194, U3 74HC86, U31 74157, U32 4017, U33 ICM7555xP, U34 4511, U35 HDSP-7503, U36 4511, U37 HDSP-7503, U4 74HC86, U44 4511, U45 74157, U46 74157, U47 HDSP-7503, U5 74HC14, U6 74HC14, U7 74147, U8 74HC04, U9 74HCT574

Commit message: finished but not checked schematic
Parts:
- removed C1, C3: 2.2μF, symbol Device:C
- removed C11, C12, C13, C14, C15, C16, C17, C18, C19, C20, C21, C22, C23, C5, C6: C, symbol Device:C
- removed C2, C4: 10nF, symbol Device:C
- removed D11, D12, D13, D14, D15, D16, D17, D18, D19, D20, D21, D22, D23, D24, D25, D26, D27, D28: 1N914, Diode_THT:D_DO-35_SOD27_P7.62mm_Horizontal, symbol Diode:1N914
- removed Q3, Q4, Q5, Q6: BC547, Package_TO_SOT_THT:TO-92_Inline, symbol Transistor_BJT:BC547
- removed R1, R179, R180, R181, R185, R196, R197, R198, R2, R209, R210, R3, R4, R5, R6, R66, R67, R68, R69, R70, R72, R74, R76, R78, R80: 10K, symbol Device:R
- removed R182, R183, R184, R237, R238, R62, R63, R64, R65, R71, R73, R75, R77, R79, R81: R, symbol Device:R
- removed R246, R247, R248, R251, R252, R253, R254, R255, R256, R257, R258, R259, R260, R261, R262, R263, R264, R265, R266, R267, R268: 330, symbol Device:R
- removed SW11, SW12, SW13, SW14, SW15, SW16, SW17, SW18, SW19, SW20, SW21, SW22, SW23: SW_Push, symbol Switch:SW_Push
- removed U18, U23, U9: 74HCT574, symbol 74xx:74HCT574
- removed unit 4 of U20
- removed unit 1 of U20
- removed unit 3 of U20
- removed unit 2 of U20
- removed unit 4 of U21
- removed unit 1 of U21
- removed unit 3 of U21
- removed unit 2 of U21
- removed unit 1 of U22
- removed U24, U25, U26, U27, U28: 74LS194, symbol 74xx:74LS194
- removed U31, U45, U46: 74157, symbol 74xx_IEEE:74157
- removed U32: 4017, symbol 4xxx:4017
- removed U33: ICM7555xP, Package_DIP:DIP-8_W7.62mm, symbol Timer:ICM7555xP
- removed U34, U36, U44: 4511, symbol 4xxx_IEEE:4511
- removed U35, U37, U47: HDSP-7503, Display_7Segment:HDSP-A151, symbol Display_Character:HDSP-7503
- removed U7: 74147, symbol 74xx_IEEE:74147
- removed unit 1 of U8
- removed unit 5 of U8
- removed unit 3 of U8
- removed unit 4 of U8
- removed unit 2 of U8
- added C10, C8: 10nF, symbol Device:C
- added C24, C25, C26, C27, C28, C29, C30, C31, C32, C33, C34, C35, C36, C37, C38: C, symbol Device:C
- added C7, C9: 2.2μF, symbol Device:C
- added D29, D30, D31, D32, D33, D34, D35, D36, D37, D38, D39, D40, D41, D42, D43, D44, D45, D46: 1N914, Diode_THT:D_DO-35_SOD27_P7.62mm_Horizontal, symbol Diode:1N914
- added Q310, Q7, Q8, Q9: BC547, Package_TO_SOT_THT:TO-92_Inline, symbol Transistor_BJT:BC547
- added R269, R270, R271, R272, R273, R274, R339, R340, R341, R342, R353, R354, R355, R356, R357, R358, R359, R360, R361, R365, R366, R367, R368, R369, R370: 10K, symbol Device:R
- added R343, R344, R345, R346, R347, R348, R349, R350, R351, R352, R362, R363, R364, R371, R372: R, symbol Device:R
- added R373, R374, R375, R376, R377, R378, R379, R380, R381, R382, R383, R384, R385, R386, R387, R388, R389, R390, R391, R392, R393: 330, symbol Device:R
- added SW24, SW25, SW26, SW27, SW28, SW29, SW30, SW31, SW32, SW33, SW34, SW35, SW36: SW_Push, symbol Switch:SW_Push
- added U48: 74147, symbol 74xx_IEEE:74147
- added U49: 74HC04, symbol 74xx:74HC04
- added U50, U51, U55: 74HCT574, symbol 74xx:74HCT574
- added U52, U53: 74HC86, symbol 74xx:74HC86
- added U54: 74HC74, symbol 74xx:74HC74
- added U56, U58, U59, U60, U61: 74LS194, symbol 74xx:74LS194
- added U57, U62, U63: 74157, symbol 74xx_IEEE:74157
- added U64: ICM7555xP, Package_DIP:DIP-8_W7.62mm, symbol Timer:ICM7555xP
- added U65: 4017, symbol 4xxx:4017
- added U66, U67, U68: 4511, symbol 4xxx_IEEE:4511
- added U69, U70, U71: HDSP-7503, Display_7Segment:HDSP-A151, symbol Display_Character:HDSP-7503
Connections:
- net +5V: now also D29.2 (A), D30.2 (A), D31.2 (A), D32.2 (A), D33.2 (A), D34.2 (A), D35.2 (A), D36.2 (A), D37.2 (A), D38.2 (A), D41.2 (A), D42.2 (A), D43.2 (A), R269.2, R270.2, R271.2, R272.2, R273.2, R274.2, R339.2, R340.2, R341.2, R342.2, R353.1, R354.1, R357.1, R359.2, R360.2, R361.2, R366.1, R367.1, R370.1, R371.1, U50.20 (VCC), U51.20 (VCC), U55.20 (VCC), U56.1 (Mr), U56.10 (S1), U56.16 (VCC), U57.16 (VCC), U58.1 (Mr), U58.10 (S1), U58.16 (VCC), U59.1 (Mr), U59.10 (S1), U59.16 (VCC), U60.1 (Mr), U60.10 (S1), U60.16 (VCC), U61.1 (Mr), U61.10 (S1), U61.16 (VCC), U62.16 (VCC), U63.16 (VCC), U64.4 (~{RST}), U64.8 (VCC), U65.16 (VDD), U66.16 (Vdd), U66.3 (~{LT}), U66.4 (~{BI}), U67.16 (Vdd), U67.3 (~{LT}), U67.4 (~{BI}), U68.16 (Vdd), U68.3 (~{LT}), U68.4 (~{BI})
- net 5V: now also U48.16 (VCC)
- net GND: now also C24.2, C25.2, C26.2, C27.2, C28.2, C29.2, C30.2, C31.2, C32.2, C33.2, C34.2, C35.2, C36.2, C37.2, C38.1, Q310.3 (E), Q7.3 (E), Q8.3 (E), Q9.3 (E), R358.2, R365.2, SW24.1, SW25.1, SW26.1, SW27.1, SW28.1, SW29.1, SW30.1, SW31.1, SW32.1, SW33.1, SW34.1, SW35.1, SW36.1, U48.8 (GND), U50.1 (OE), U50.10 (GND), U51.1 (OE), U51.10 (GND), U54.2 (D), U54.3 (C), U55.1 (OE), U55.10 (GND), U56.8 (GND), U57.15 (~{EN}), U57.8 (GND), U58.8 (GND), U59.8 (GND), U60.8 (GND), U61.7 (Dsl), U61.8 (GND), U62.15 (~{EN}), U62.8 (GND), U63.15 (~{EN}), U63.8 (GND), U64.1 (GND), U65.13 (CKEN), U65.8 (VSS), U66.5 (~{EL}), U66.8 (Vss), U67.5 (~{EL}), U67.8 (Vss), U68.5 (~{EL}), U68.8 (Vss), U69.1 (CC), U69.6 (CC), U69.7 (DP), U70.1 (CC), U70.6 (CC), U70.7 (DP), U71.1 (CC), U71.6 (CC), U71.7 (DP)
- new net: R273.1, R347.1, SW28.2
- new net: C29.1, D34.1 (K), R348.2, U48.3 (~{E6})
- new net: R376.1, U66.10 (Qd)
- new net: R376.2, U69.5 (D)
- new net: R341.1, R351.1, SW32.2
- new net: C32.1, D37.1 (K), R351.2, U48.10 (~{E9})
- new net: R371.2, R372.1, U64.7 (DISCH)
- new net: R269.1, R343.1, SW24.2
- new net: R274.1, R348.1, SW29.2
- new net: R378.1, U66.15 (Qf)
- new net: R378.2, U69.2 (F)
- new net: Q7.2 (B), R355.1, R356.1
- new net: D39.2 (A), Q8.1 (C), R356.2, R357.2
- new net: C8.2, R355.2
- new net: R361.1, R364.1, SW36.2
- new net: U57.4 (Qa), U58.3 (P0)
- new net: U57.7 (Qb), U58.4 (P1)
- new net: U57.12 (Qc), U58.5 (P2)
- new net: U57.9 (Qd), U58.6 (P3)
- new net: U56.9 (S0), U58.9 (S0), U59.9 (S0), U60.9 (S0), U61.9 (S0), U65.3 (Q0)
- new net: C9.1, Q310.2 (B), R367.2
- new net: C26.1, D31.1 (K), R345.2, U48.13 (~{E3})
- new net: R377.1, U66.9 (Qe)
- new net: R377.2, U69.4 (E)
- new net: R270.1, R344.1, SW25.2
- new net: C10.1, C36.1, D43.1 (K), R364.2, U65.15 (Reset)
- new net: U48.7 (~{S1}), U49.3
- new net: R339.1, R349.1, SW30.2
- new net: C30.1, D35.1 (K), R349.2, U48.4 (~{E7})
- new net: C28.1, D33.1 (K), R347.2, U48.2 (~{E5})
- new net: U51.12 (Q7), U53.12
- new net: C7.2, Q7.1 (C), R353.2
- new net: C27.1, D32.1 (K), R346.2, U48.1 (~{E4})
- new net: U51.16 (Q3), U52.12
- new net: R393.1, U68.14 (Qg)
- new net: R393.2, U71.3 (G)
- new net: C7.1, Q8.2 (B), R354.2
- new net: U51.14 (Q5), U53.9
- new net: U48.6 (~{S2}), U49.5
- new net: C24.1, D29.1 (K), R343.2, U48.11 (~{E1})
- new net: R384.1, U67.9 (Qe)
- new net: R384.2, U70.4 (E)
- new net: C10.2, R368.2
- new net: R392.1, U68.15 (Qf)
- new net: R392.2, U71.2 (F)
- new net: R272.1, R346.1, SW27.2
- new net: R381.1, U67.12 (Qb)
- new net: R381.2, U70.9 (B)
- new net: R388.1, U68.12 (Qb)
- new net: R388.2, U71.9 (B)
- new net: R373.2, U69.10 (A)
- new net: R379.2, U69.3 (G)
- new net: R375.2, U69.8 (C)
- new net: R374.2, U69.9 (B)
- new net: C37.1, C38.2, R372.2, U64.2 (TRIG), U64.5 (CONT), U64.6 (THRES)
- new net: Q9.1 (C), R366.2
- new net: Q9.2 (B), R368.1, R369.1
- new net: R387.1, U68.13 (Qa)
- new net: R387.2, U71.10 (A)
- new net: R391.2, U71.4 (E)
- new net: R390.2, U71.5 (D)
- new net: R389.2, U71.8 (C)
- new net: R342.1, R352.1, SW33.2
- new net: U51.15 (Q4), U53.1
- new net: U59.3 (P0), U62.4 (Qa)
- new net: U59.4 (P1), U62.7 (Qb)
- new net: U59.5 (P2), U62.12 (Qc)
- new net: U59.6 (P3), U62.9 (Qd)
- new net: U59.7 (Dsl), U60.12 (Q3)
- new net: R375.1, U66.11 (Qc)
- new net: R360.1, R363.1, SW35.2
- new net: R390.1, U68.10 (Qd)
- new net: R380.2, U70.10 (A)
- new net: R385.2, U70.2 (F)
- new net: R386.2, U70.3 (G)
- new net: R383.2, U70.5 (D)
- new net: R382.2, U70.8 (C)
- new net: U55.15 (Q4), U60.3 (P0)
- new net: U55.14 (Q5), U60.4 (P1)
- new net: U55.13 (Q6), U60.5 (P2)
- new net: U55.12 (Q7), U60.6 (P3)
- new net: U60.7 (Dsl), U61.12 (Q3)
- new net: R382.1, U67.11 (Qc)
- new net: R359.1, R362.1, SW34.2
- new net: D46.2 (A), Q310.1 (C), R369.2, R370.2, U55.11 (Cp)
- new net: R379.1, U66.14 (Qg)
- new net: R374.1, U66.12 (Qb)
- new net: U48.9 (~{S0}), U49.1
- new net: C33.1, D38.1 (K), R352.2, U49.11
- new net: U56.5 (P2), U63.12 (Qc)
- new net: U56.3 (P0), U63.4 (Qa)
- new net: U56.4 (P1), U63.7 (Qb)
- new net: U56.6 (P3), U63.9 (Qd)
- new net: R340.1, R350.1, SW31.2
- new net: R391.1, U68.9 (Qe)
- new net: U51.19 (Q0), U52.1
- new net: C25.1, D30.1 (K), R344.2, U48.12 (~{E2})
- new net: C31.1, D36.1 (K), R350.2, U48.5 (~{E8})
- new net: U51.17 (Q2), U52.4
- new net: R385.1, U67.15 (Qf)
- new net: R271.1, R345.1, SW26.2
- new net: R389.1, U68.11 (Qc)
- new net: R373.1, U66.13 (Qa)
- new net: U51.13 (Q6), U53.4
- new net: R383.1, U67.10 (Qd)
- new net: R386.1, U67.14 (Qg)
- new net: U48.14 (~{S3}), U49.9
- new net: U55.16 (Q3), U61.6 (P3)
- new net: U55.17 (Q2), U61.5 (P2)
- new net: U55.18 (Q1), U61.4 (P1)
- new net: U55.19 (Q0), U61.3 (P0)
- new net: U51.18 (Q1), U52.9
- new net: R380.1, U67.13 (Qa)
- new net =: D39.1 (K), D40.1 (K), D46.1 (K), R358.1, U50.11 (Cp)
- new net AND16/IN_A: U59.14 (Q1), U62.5 (I0b), U67.1 (DB)
- new net AND16/IN_B: U59.13 (Q2), U62.14 (I0c), U67.2 (DC)
- new net AND17/IN_A: U55.8 (D6)
- new net AND18/IN_A: U55.9 (D7)
- new net AND19/IN_A: U55.7 (D5)
- new net AND20/IN_A: U55.6 (D4)
- new net AND21/IN_B: U64.3 (OUT)
- new net AND21/OUTPUT: U56.11 (Cp), U58.11 (Cp), U59.11 (Cp), U60.11 (Cp), U61.11 (Cp), U65.14 (CLK)
- new net AND22/IN_A: U56.14 (Q1), U63.14 (I0c), U63.5 (I0b), U68.1 (DB)
- new net AND22/IN_B: U56.13 (Q2), U68.2 (DC)
- new net AND23/IN_A: U55.4 (D2)
- new net AND24/IN_A: U55.5 (D3)
- new net AND25/IN_A: U55.2 (D0), U55.3 (D1)
- new net AND27/IN_A: C34.1, D41.1 (K), R362.2, U54.1 (~{R})
- new net AND27/IN_B: C35.1, D42.1 (K), R363.2, R365.1, U54.4 (~{S})
- new net AND28/IN_B: U59.15 (Q0), U62.2 (I0a), U67.7 (DA)
- new net AND29/IN_A: U57.14 (I0c), U58.13 (Q2), U66.2 (DC)
- new net AND29/IN_B: U57.5 (I0b), U58.14 (Q1), U66.1 (DB)
- new net AND30/IN_B: U56.15 (Q0), U63.2 (I0a), U68.7 (DA)
- new net AND31/IN_B: U57.2 (I0a), U58.15 (Q0), U66.7 (DA)
- new net FULL_ADDER28/IN_B: U52.8
- new net FULL_ADDER29/IN_B: U52.6
- new net FULL_ADDER30/IN_B: U52.11
- new net FULL_ADDER31/IN_B: U53.3
- new net FULL_ADDER40/IN_B: U53.8
- new net FULL_ADDER41/IN_B: U53.6
- new net FULL_ADDER42/IN_B: U53.11
- new net FULL_ADDER59/IN_B: U52.3
- new net FULL_ADDER59/IN_C: U52.10, U52.13, U52.2, U52.5, U53.10, U53.13, U53.2, U53.5, U54.5 (Q)
- new net FULL_ADDER60/OUT_S: U62.3 (I1a)
- new net FULL_ADDER61/OUT_S: U62.6 (I1b)
- new net FULL_ADDER62/OUT_S: U62.13 (I1c)
- new net FULL_ADDER63/IN_A: U58.7 (Dsl), U59.12 (Q3), U62.11 (I0d), U67.6 (DD)
- new net FULL_ADDER63/OUT_S: U62.10 (I1d)
- new net FULL_ADDER64/OUT_S: U63.3 (I1a)
- new net FULL_ADDER65/OUT_S: U63.6 (I1b)
- new net FULL_ADDER66/OUT_S: U63.13 (I1c)
- new net FULL_ADDER67/IN_A: U56.12 (Q3), U63.11 (I0d), U68.6 (DD)
- new net FULL_ADDER67/OUT_S: U63.10 (I1d)
- new net FULL_ADDER68/OUT_S: U57.3 (I1a)
- new net FULL_ADDER69/OUT_S: U57.6 (I1b)
- new net FULL_ADDER70/OUT_S: U57.13 (I1c)
- new net FULL_ADDER71/IN_A: U56.7 (Dsl), U57.11 (I0d), U58.12 (Q3), U66.6 (DD)
- new net FULL_ADDER71/OUT_S: U57.10 (I1d)
- new net OR11/IN_A: U49.6
- new net OR11/IN_B: U49.8
- new net OR13/IN_B: U49.10
- new net OR13/OUTPUT: C8.1
- new net OR16/OUTPUT: U62.1 (A/B)
- new net OR18/OUTPUT: U63.1 (A/B)
- new net OR19/OUTPUT: U57.1 (A/B)
- new net OR5/IN_A: U49.2
- new net OR5/IN_B: U49.4
- new net U50_D0: U50.2 (D0)
- new net U50_D1: U50.3 (D1)
- new net U50_D2: U50.4 (D2)
- new net U50_D3: U50.5 (D3)
- new net U50_D4: U50.6 (D4)
- new net U50_D5: U50.7 (D5)
- new net U50_D6: U50.8 (D6)
- new net U50_D7: U50.9 (D7)
- new net U50_Q0: U50.12 (Q7), U51.9 (D7)
- new net U50_Q1: U50.13 (Q6), U51.8 (D6)
- new net U50_Q2: U50.14 (Q5), U51.7 (D5)
- new net U50_Q3: U50.15 (Q4), U51.6 (D4)
- new net U50_Q4: U50.16 (Q3), U51.5 (D3)
- new net U50_Q5: U50.17 (Q2), U51.4 (D2)
- new net U50_Q6: U50.18 (Q1), U51.3 (D1)
- new net U50_Q7: U50.19 (Q0), U51.2 (D0)
- new net btns: D40.2 (A), D44.1 (K), D45.1 (K), U51.11 (Cp)
- new net not3/OUTPUT: D44.2 (A)
- new net not4/OUTPUT: D45.2 (A)
- new net not5/INPUT: U65.11 (Q9)
Other:
- removed sheet AND
- removed sheet AND1
- removed sheet AND10
- removed sheet AND11
- removed sheet AND12
- removed sheet AND13
- removed sheet AND14
- removed sheet AND15
- removed sheet AND2
- removed sheet AND3
- removed sheet AND4
- removed sheet AND5
- removed sheet AND6
- removed sheet AND7
- removed sheet AND8
- removed sheet AND9
- removed sheet FULL_ADDER
- removed sheet FULL_ADDER1
- removed sheet FULL_ADDER10
- removed sheet FULL_ADDER11
- removed sheet FULL_ADDER12
- removed sheet FULL_ADDER13
- removed sheet FULL_ADDER14
- removed sheet FULL_ADDER15
- removed sheet FULL_ADDER16
- removed sheet FULL_ADDER17
- removed sheet FULL_ADDER18
- removed sheet FULL_ADDER19
- removed sheet FULL_ADDER2
- removed sheet FULL_ADDER20
- removed sheet FULL_ADDER21
- removed sheet FULL_ADDER22
- removed sheet FULL_ADDER23
- removed sheet FULL_ADDER24
- removed sheet FULL_ADDER25
- removed sheet FULL_ADDER26
- removed sheet FULL_ADDER27
- removed sheet FULL_ADDER3
- removed sheet FULL_ADDER32
- removed sheet FULL_ADDER33
- removed sheet FULL_ADDER34
- removed sheet FULL_ADDER35
- removed sheet FULL_ADDER36
- removed sheet FULL_ADDER37
- removed sheet FULL_ADDER38
- removed sheet FULL_ADDER39
- removed sheet FULL_ADDER4
- removed sheet FULL_ADDER5
- removed sheet FULL_ADDER6
- removed sheet FULL_ADDER7
- removed sheet FULL_ADDER8
- removed sheet FULL_ADDER9
- removed sheet OR
- removed sheet OR1
- removed sheet OR10
- removed sheet OR2
- removed sheet OR3
- removed sheet OR4
- removed sheet OR6
- removed sheet OR7
- removed sheet OR8
- removed sheet OR9
- removed sheet not
- removed sheet not1
- removed sheet not2
- added sheet AND16 (AND_gate.kicad_sch)
- added sheet AND17 (AND_gate.kicad_sch)
- added sheet AND18 (AND_gate.kicad_sch)
- added sheet AND19 (AND_gate.kicad_sch)
- added sheet AND20 (AND_gate.kicad_sch)
- added sheet AND21 (AND_gate.kicad_sch)
- added sheet AND22 (AND_gate.kicad_sch)
- added sheet AND23 (AND_gate.kicad_sch)
- added sheet AND24 (AND_gate.kicad_sch)
- added sheet AND25 (AND_gate.kicad_sch)
- added sheet AND26 (AND_gate.kicad_sch)
- added sheet AND27 (AND_gate.kicad_sch)
- added sheet AND28 (AND_gate.kicad_sch)
- added sheet AND29 (AND_gate.kicad_sch)
- added sheet AND30 (AND_gate.kicad_sch)
- added sheet AND31 (AND_gate.kicad_sch)
- added sheet FULL_ADDER28 (full_adder.kicad_sch)
- added sheet FULL_ADDER29 (full_adder.kicad_sch)
- added sheet FULL_ADDER30 (full_adder.kicad_sch)
- added sheet FULL_ADDER31 (full_adder.kicad_sch)
- added sheet FULL_ADDER40 (full_adder.kicad_sch)
- added sheet FULL_ADDER41 (full_adder.kicad_sch)
- added sheet FULL_ADDER42 (full_adder.kicad_sch)
- added sheet FULL_ADDER43 (full_adder.kicad_sch)
- added sheet FULL_ADDER44 (full_adder.kicad_sch)
- added sheet FULL_ADDER45 (full_adder.kicad_sch)
- added sheet FULL_ADDER46 (full_adder.kicad_sch)
- added sheet FULL_ADDER47 (full_adder.kicad_sch)
- added sheet FULL_ADDER48 (full_adder.kicad_sch)
- added sheet FULL_ADDER49 (full_adder.kicad_sch)
- added sheet FULL_ADDER50 (full_adder.kicad_sch)
- added sheet FULL_ADDER51 (full_adder.kicad_sch)
- added sheet FULL_ADDER52 (full_adder.kicad_sch)
- added sheet FULL_ADDER53 (full_adder.kicad_sch)
- added sheet FULL_ADDER54 (full_adder.kicad_sch)
- added sheet FULL_ADDER55 (full_adder.kicad_sch)
- added sheet FULL_ADDER56 (full_adder.kicad_sch)
- added sheet FULL_ADDER57 (full_adder.kicad_sch)
- added sheet FULL_ADDER58 (full_adder.kicad_sch)
- added sheet FULL_ADDER59 (full_adder.kicad_sch)
- added sheet FULL_ADDER60 (full_adder.kicad_sch)
- added sheet FULL_ADDER61 (full_adder.kicad_sch)
- added sheet FULL_ADDER62 (full_adder.kicad_sch)
- added sheet FULL_ADDER63 (full_adder.kicad_sch)
- added sheet FULL_ADDER64 (full_adder.kicad_sch)
- added sheet FULL_ADDER65 (full_adder.kicad_sch)
- added sheet FULL_ADDER66 (full_adder.kicad_sch)
- added sheet FULL_ADDER67 (full_adder.kicad_sch)
- added sheet FULL_ADDER68 (full_adder.kicad_sch)
- added sheet FULL_ADDER69 (full_adder.kicad_sch)
- added sheet FULL_ADDER70 (full_adder.kicad_sch)
- added sheet FULL_ADDER71 (full_adder.kicad_sch)
- added sheet OR11 (OR_gate.kicad_sch)
- added sheet OR12 (OR_gate.kicad_sch)
- added sheet OR13 (OR_gate.kicad_sch)
- added sheet OR14 (OR_gate.kicad_sch)
- added sheet OR15 (OR_gate.kicad_sch)
- added sheet OR16 (OR_gate.kicad_sch)
- added sheet OR17 (OR_gate.kicad_sch)
- added sheet OR18 (OR_gate.kicad_sch)
- added sheet OR19 (OR_gate.kicad_sch)
- added sheet OR5 (OR_gate.kicad_sch)
- added sheet not3 (not.kicad_sch)
- added sheet not4 (not.kicad_sch)
- added sheet not5 (not.kicad_sch)
