File: AND_gate.kicad_sch (KiCad schematic)
At the start: 5 parts, among them Q31 DTC114E, Q32 DTC114E, Q33 DTC114E

Commit message: 0 errors + 0 warnings
Parts:
- removed Q31, Q32: DTC114E, symbol Transistor_BJT:DTC114E
- added Q229, Q34: DTC114E, Package_TO_SOT_SMD:SOT-23-3, symbol Transistor_BJT:DTC114E
- Q33: footprint (none) -> Package_TO_SOT_SMD:SOT-23-3
- R21, R22: footprint (none) -> Resistor_SMD:R_0603_1608Metric
Connections:
- net GND: now also Q229.2 (E)
- net IN_A: now also Q34.1 (B)
- net IN_B: now also Q229.1 (B)
- net at Q33.1 (B), R21.2: now also Q34.3 (C)
- new net: Q229.3 (C), Q34.2 (E)
