File: full_adder.kicad_sch (KiCad schematic)
At the start: 0 parts

Commit message: 0 errors + 0 warnings
Other:
- sheet HALF_ADDER renamed HALF_ADDER3
- sheet HALF_ADDER1 renamed HALF_ADDER2
Changed lines of the file:
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@@
-	(wire
-		(pts
-			(xy 19.1262 0.0762) (xy 22.9362 0.0762)
-		)
-		(stroke
-			(width 0)
-			(type default)
-		)
-	)
 	(wire
 		(pts
@@
 	(wire
 		(pts
-			(xy 22.9362 0.0762) (xy 22.9362 62.3062)
-		)
-		(stroke
-			(width 0)
-			(type default)
-		)
-	)
-	(wire
-		(pts
 			(xy 91.44 91.44) (xy 99.06 91.44)
 		)
@@
 		(pts
 			(xy 152.4 93.98) (xy 153.67 93.98)
-		)
-		(stroke
-			(width 0)
-			(type default)
-		)
-	)
-	(wire
-		(pts
-			(xy 22.9362 62.3062) (xy 0.0762 62.3062)
 		)
 		(stroke
@@
 			(color 0 0 0 0)
 		)
-		(property "Sheetname" "HALF_ADDER1"
+		(property "Sheetname" "HALF_ADDER2"
 			(at 99.06 81.8384 0)
 			(show_name no)
@@
 			(color 0 0 0 0)
 		)
-		(property "Sheetname" "HALF_ADDER"
+		(property "Sheetname" "HALF_ADDER3"
 			(at 120.65 81.8384 0)
 			(show_name no)
