File: half_Adder.kicad_sch (KiCad schematic)
At the start: 0 parts

Commit message: 0 errors + 0 warnings
Changed lines of the file:
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@@
-	(wire
-		(pts
-			(xy 0.0762 0.0762) (xy 0.0762 7.6962)
-		)
-		(stroke
-			(width 0)
-			(type default)
-		)
-	)
 	(wire
 		(pts
@@
 		)
 		(stroke
-			(width 0)
-			(type default)
-		)
-	)
-	(wire
-		(pts
-			(xy 0.0762 7.6962) (xy 19.1262 7.6962)
-		)
-		(stroke
