File: not.kicad_sch (KiCad schematic)
At the start: 2 parts, among them Q239 DTC114E

Commit message: 0 errors + 0 warnings
Parts:
- Q239: footprint (none) -> Package_TO_SOT_SMD:SOT-23-3
- R186: footprint (none) -> Resistor_SMD:R_0603_1608Metric
Changed lines of the file:
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@@
-		)
-	)
-	(label "OUTPUT (OR)"
-		(at 152.4 92.71 0)
-		(effects
-			(font
-				(size 1.27 1.27)
-			)
-			(justify left bottom)
 		)
 	)
@@
 					(unit 1)
 				)
+				(path "/43e6f3ed-0436-432c-97f0-d30a4f4230c3/57ecb8c8-ce7d-4e03-9fbb-3e4caa8b261c"
+					(reference "#PWR0783")
+					(unit 1)
+				)
+				(path "/43e6f3ed-0436-432c-97f0-d30a4f4230c3/644dfea1-fbbe-4f00-9a35-31e3571483b6"
+					(reference "#PWR0779")
+					(unit 1)
+				)
+				(path "/43e6f3ed-0436-432c-97f0-d30a4f4230c3/646dcff9-da4f-43e2-bb94-c5515a400505"
+					(reference "#PWR0785")
+					(unit 1)
+				)
+				(path "/43e6f3ed-0436-432c-97f0-d30a4f4230c3/84f69074-509c-4f33-a663-ddefc8434239"
+					(reference "#PWR0777")
+					(unit 1)
+				)
+				(path "/43e6f3ed-0436-432c-97f0-d30a4f4230c3/88bd5815-8b89-4c1e-ba8c-20ae8b4112f9"
+					(reference "#PWR0781")
+					(unit 1)
+				)
 				(path "/43e6f3ed-0436-432c-97f0-d30a4f4230c3/ee4f650b-d7f3-4c56-b231-40b61ce91f3c"
 					(reference "#PWR0431")
@@
 			)
 		)
-		(property "Footprint" ""
+		(property "Footprint" "Resistor_SMD:R_0603_1608Metric"
 			(at 146.812 82.55 90)
 			(hide yes)
@@
 				(path "/43e6f3ed-0436-432c-97f0-d30a4f4230c3/4d747a09-e608-492c-8ace-d75dcdfbdcd5"
 					(reference "R186")
+					(unit 1)
+				)
+				(path "/43e6f3ed-0436-432c-97f0-d30a4f4230c3/57ecb8c8-ce7d-4e03-9fbb-3e4caa8b261c"
+					(reference "R272")
+					(unit 1)
+				)
+				(path "/43e6f3ed-0436-432c-97f0-d30a4f4230c3/644dfea1-fbbe-4f00-9a35-31e3571483b6"
+					(reference "R270")
+					(unit 1)
+				)
+				(path "/43e6f3ed-0436-432c-97f0-d30a4f4230c3/646dcff9-da4f-43e2-bb94-c5515a400505"
+					(reference "R273")
+					(unit 1)
+				)
+				(path "/43e6f3ed-0436-432c-97f0-d30a4f4230c3/84f69074-509c-4f33-a663-ddefc8434239"
+					(reference "R269")
+					(unit 1)
+				)
+				(path "/43e6f3ed-0436-432c-97f0-d30a4f4230c3/88bd5815-8b89-4c1e-ba8c-20ae8b4112f9"
+					(reference "R271")
 					(unit 1)
 				)
@@
 			)
 		)
-		(property "Footprint" ""
+		(property "Footprint" "Package_TO_SOT_SMD:SOT-23-3"
 			(at 146.05 99.06 0)
 			(hide yes)
@@
 				(path "/43e6f3ed-0436-432c-97f0-d30a4f4230c3/4d747a09-e608-492c-8ace-d75dcdfbdcd5"
 					(reference "Q239")
+					(unit 1)
+				)
+				(path "/43e6f3ed-0436-432c-97f0-d30a4f4230c3/57ecb8c8-ce7d-4e03-9fbb-3e4caa8b261c"
+					(reference "Q251")
+					(unit 1)
+				)
+				(path "/43e6f3ed-0436-432c-97f0-d30a4f4230c3/644dfea1-fbbe-4f00-9a35-31e3571483b6"
+					(reference "Q245")
+					(unit 1)
+				)
+				(path "/43e6f3ed-0436-432c-97f0-d30a4f4230c3/646dcff9-da4f-43e2-bb94-c5515a400505"
+					(reference "Q256")
+					(unit 1)
+				)
+				(path "/43e6f3ed-0436-432c-97f0-d30a4f4230c3/84f69074-509c-4f33-a663-ddefc8434239"
+					(reference "Q242")
+					(unit 1)
+				)
+				(path "/43e6f3ed-0436-432c-97f0-d30a4f4230c3/88bd5815-8b89-4c1e-ba8c-20ae8b4112f9"
+					(reference "Q248")
 					(unit 1)
 				)
@@
 					(unit 1)
 				)
+				(path "/43e6f3ed-0436-432c-97f0-d30a4f4230c3/57ecb8c8-ce7d-4e03-9fbb-3e4caa8b261c"
+					(reference "#PWR0782")
+					(unit 1)
+				)
+				(path "/43e6f3ed-0436-432c-97f0-d30a4f4230c3/644dfea1-fbbe-4f00-9a35-31e3571483b6"
+					(reference "#PWR0778")
+					(unit 1)
+				)
+				(path "/43e6f3ed-0436-432c-97f0-d30a4f4230c3/646dcff9-da4f-43e2-bb94-c5515a400505"
+					(reference "#PWR0784")
+					(unit 1)
+				)
+				(path "/43e6f3ed-0436-432c-97f0-d30a4f4230c3/84f69074-509c-4f33-a663-ddefc8434239"
+					(reference "#PWR0776")
+					(unit 1)
+				)
+				(path "/43e6f3ed-0436-432c-97f0-d30a4f4230c3/88bd5815-8b89-4c1e-ba8c-20ae8b4112f9"
+					(reference "#PWR0780")
+					(unit 1)
+				)
