File: untitled.kicad_sch (KiCad schematic)
At the start: 1 part, among them U4 74HC86

Commit message: 0 errors + 0 warnings
Parts:
- U4: footprint (none) -> Package_SO:TSSOP-14_4.4x5mm_P0.65mm
Changed lines of the file:
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@@
 			)
 		)
-		(property "Footprint" ""
+		(property "Footprint" "Package_SO:TSSOP-14_4.4x5mm_P0.65mm"
 			(at 115.57 105.41 0)
 			(hide yes)
