File: calc.kicad_sch (KiCad schematic)
At the start: 145 parts, among them Q3 BC547, Q4 BC547, Q5 BC547, Q6 BC547, SW11 SW_Push, SW12 SW_Push, SW13 SW_Push, SW14 SW_Push, SW15 SW_Push, SW16 SW_Push, SW17 SW_Push, SW18 SW_Push, SW19 SW_Push, SW20 SW_Push, SW21 SW_Push, SW22 SW_Push, SW23 SW_Push, U1 74HC86, U18 74HCT574, U2 74HC86, U20 74HC86, U21 74HC86, U22 74HC74, U23 74HCT574, U24 74LS194, U25 74LS194, U26 74LS194, U27 74LS194, U28 74LS194, U3 74HC86, U31 74157, U32 4017, U33 ICM7555xP, U34 4511, U35 HDSP-7503, U36 4511, U37 HDSP-7503, U4 74HC86, U44 4511, U45 74157, U46 74157, U47 HDSP-7503, U5 74HC14, U6 74HC14, U7 74147, U8 74HC04, U9 74HCT574

Commit message: 0 errors + 0 warnings
Parts:
- removed U5, U6: 74HC14, symbol 74xx:74HC14
- removed U8: 74HC04, symbol 74xx:74HC04
- added C7: 0.1µF, Capacitor_SMD:C_0603_1608Metric, symbol Device:C
- added C8: 10µF, Capacitor_SMD:C_0603_1608Metric, symbol Device:C
- added J1: Conn_01x02_Pin, Connector_PinHeader_2.54mm:PinHeader_1x02_P2.54mm_Vertical, symbol Connector:Conn_01x02_Pin
- added J2: Conn_01x03_Pin, Connector_PinHeader_2.54mm:PinHeader_1x03_P2.54mm_Vertical, symbol Connector:Conn_01x03_Pin
- added U10, U11, U12, U13, U14, U15, U16, U17, U19, U29, U30, U38, U39, U40, U41, U42: 74HC86, Package_SO:TSSOP-14_4.4x5mm_P0.65mm, symbol 74xx:74HC86
- added unit 1 of U4
- added U43, U48, U49: 74HC86, symbol 74xx:74HC86
- added U56: L7805, Connector_PinHeader_2.54mm:PinHeader_1x03_P2.54mm_Vertical, symbol Regulator_Linear:L7805
- C1, C2, C3, C4: footprint (none) -> Capacitor_SMD:C_0603_1608Metric
- C11, C12, C13, C14, C15, C16, C17, C18, C19, C20, C21, C22, C23, C6: value C -> 1µF; footprint (none) -> Capacitor_SMD:C_0603_1608Metric
- C5: value C -> 100nF; footprint (none) -> Capacitor_SMD:C_0603_1608Metric
- R1, R179, R180, R181, R185, R196, R197, R198, R2, R209, R210, R3, R4, R5, R6, R66, R67, R68, R69, R70, R72, R74, R76, R78, R80: footprint (none) -> Resistor_SMD:R_0603_1608Metric
- R182, R183, R184, R237, R62, R63, R64, R65, R71, R73, R75, R77, R79, R81: value R -> 10K; footprint (none) -> Resistor_SMD:R_0603_1608Metric
- R238: value R -> 47K; footprint (none) -> Resistor_SMD:R_0603_1608Metric
- R246, R247, R248, R251, R252, R253, R254, R255, R256, R257, R258, R259, R260, R261, R262, R263, R264, R265, R266, R267, R268: value 330 -> 330Ω; footprint (none) -> Resistor_SMD:R_0603_1608Metric
- SW11, SW12, SW13, SW14, SW15, SW16, SW17, SW18, SW19, SW20, SW21, SW22, SW23: footprint (none) -> Button_Switch_Keyboard:SW_Cherry_MX_1.00u_PCB
- U1, U2, U20, U21, U3, U4: footprint (none) -> Package_SO:TSSOP-14_4.4x5mm_P0.65mm
- U18, U23, U9: footprint (none) -> Package_DIP:DIP-20_W7.62mm_LongPads
- U22: footprint (none) -> Package_DIP:DIP-14_W10.16mm_LongPads
- U24, U25, U26, U27, U28, U31, U32, U34, U36, U44, U45, U46, U7: footprint (none) -> Package_DIP:DIP-16_W10.16mm_LongPads
Connections:
- net 5V is gone; now on net +5V: U1.14 (VCC), U2.14 (VCC), U20.14 (VCC), U21.14 (VCC), U22.14 (VCC), U3.14 (VCC), U4.14 (VCC), U7.16 (VCC)
- net +5V: now also U22.10 (~{S}), U22.13 (~{R}), C7.1, U10.14 (VCC), U11.14 (VCC), U12.14 (VCC), U13.14 (VCC), U14.14 (VCC), U15.14 (VCC), U16.14 (VCC), U17.14 (VCC), U19.14 (VCC), U29.14 (VCC), U30.14 (VCC), U38.14 (VCC), U39.14 (VCC), U40.14 (VCC), U41.14 (VCC), U42.14 (VCC), U43.14 (VCC), U48.14 (VCC), U49.14 (VCC), U56.3 (OUT)
- net AND10/IN_A: no longer U23.2 (D0), U23.3 (D1)
- net GND: now also U22.11 (C), U22.12 (D), U24.2 (Dsr), U25.2 (Dsr), U26.2 (Dsr), U27.2 (Dsr), U28.2 (Dsr), C7.2, C8.2, J1.1 (Pin_1), U10.7 (GND), U11.7 (GND), U12.7 (GND), U13.7 (GND), U14.7 (GND), U15.7 (GND), U16.7 (GND), U17.7 (GND), U19.7 (GND), U29.7 (GND), U30.7 (GND), U38.7 (GND), U39.7 (GND), U40.7 (GND), U41.7 (GND), U42.7 (GND), U43.7 (GND), U48.7 (GND), U49.7 (GND), U56.2 (GND)
- net at Q5.1 (C), R185.2: now also C3.2
- net not7/INPUT: now reaches U7.9 (~{S0})
- net not3/INPUT: now reaches C17.1, D17.1 (K), R75.2
- net not5/INPUT: now reaches U7.6 (~{S2})
- net not4/INPUT: now reaches U7.14 (~{S3})
- net not6/INPUT: now reaches U7.7 (~{S1})
- new net: J1.2 (Pin_2), J2.2 (Pin_2)
- new net: C8.1, J2.3 (Pin_3), U56.1 (IN)
- new net AND9/IN_A: U23.3 (D1)
- new net FULL_ADDER23/OUT_S: U23.2 (D0)
- no-connect marks 1 -> 85
Other:
- added sheet not3 (not.kicad_sch)
- added sheet not4 (not.kicad_sch)
- added sheet not5 (not.kicad_sch)
- added sheet not6 (not.kicad_sch)
- added sheet not7 (not.kicad_sch)
- moved on the sheet: U20E, U21E, U22B, U22C, U2E, U3E, U4E

Commit message: footprints
Parts:
- U29, U30, U38, U39, U4, U42, U43, U48, U49: footprint (none) -> Package_SO:TSSOP-14_4.4x5mm_P0.65mm
Other:
- moved on the sheet: U22B
Changed lines of the file:
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@@
 	(generator "eeschema")
 	(generator_version "10.0")
-	(paper "User" 1270 1270)
+	(paper "User" 1270 762)
 	(text "-"
 		(exclude_from_sim no)
@@
 	)
 	(no_connect
-		(at 1205.23 1212.85)
+		(at 830.58 72.39)
 	)
 	(no_connect
@@
 	)
 	(no_connect
-		(at 1205.23 1207.77)
+		(at 830.58 67.31)
 	)
 	(no_connect
@@
 	(wire
 		(pts
-			(xy 1197.61 1221.74) (xy 1200.15 1221.74)
+			(xy 822.96 81.28) (xy 825.5 81.28)
 		)
 		(stroke
@@
 	(wire
 		(pts
-			(xy 1187.45 1207.77) (xy 1189.99 1207.77)
+			(xy 812.8 67.31) (xy 815.34 67.31)
 		)
 		(stroke
@@
 	(wire
 		(pts
-			(xy 1197.61 1217.93) (xy 1197.61 1221.74)
+			(xy 822.96 77.47) (xy 822.96 81.28)
 		)
 		(stroke
@@
 			)
 		)
-		(property "Footprint" ""
+		(property "Footprint" "Package_SO:TSSOP-14_4.4x5mm_P0.65mm"
 			(at 668.02 45.72 0)
 			(hide yes)
@@
 			)
 		)
-		(property "Footprint" ""
+		(property "Footprint" "Package_SO:TSSOP-14_4.4x5mm_P0.65mm"
 			(at 712.47 99.06 0)
 			(hide yes)
@@
 	(symbol
 		(lib_id "power:GND")
-		(at 1189.99 1210.31 0)
+		(at 815.34 69.85 0)
 		(unit 1)
 		(body_style 1)
@@
 		(fields_autoplaced yes)
 		(property "Reference" "#PWR0555"
-			(at 1189.99 1216.66 0)
+			(at 815.34 76.2 0)
 			(hide yes)
 			(show_name no)
@@
 		)
 		(property "Value" "GND"
-			(at 1189.99 1215.39 0)
+			(at 815.34 74.93 0)
 			(show_name no)
 			(do_not_autoplace no)
@@
 		)
 		(property "Footprint" ""
-			(at 1189.99 1210.31 0)
+			(at 815.34 69.85 0)
 			(hide yes)
 			(show_name no)
@@
 		)
 		(property "Datasheet" ""
-			(at 1189.99 1210.31 0)
+			(at 815.34 69.85 0)
 			(hide yes)
 			(show_name no)
@@
 		)
 		(property "Description" "Power symbol creates a global label with name \"GND\" , ground"
-			(at 1189.99 1210.31 0)
+			(at 815.34 69.85 0)
 			(hide yes)
 			(show_name no)
@@
 			)
 		)
-		(property "Footprint" ""
+		(property "Footprint" "Package_SO:TSSOP-14_4.4x5mm_P0.65mm"
 			(at 750.57 64.77 0)
 			(hide yes)
@@
 	(symbol
 		(lib_id "power:+5V")
-		(at 1197.61 1202.69 0)
+		(at 822.96 62.23 0)
 		(unit 1)
 		(body_style 1)
@@
 		(fields_autoplaced yes)
 		(property "Reference" "#PWR0557"
-			(at 1197.61 1206.5 0)
+			(at 822.96 66.04 0)
 			(hide yes)
 			(show_name no)
@@
 		)
 		(property "Value" "+5V"
-			(at 1197.61 1197.61 0)
+			(at 822.96 57.15 0)
 			(show_name no)
 			(do_not_autoplace no)
@@
 		)
 		(property "Footprint" ""
-			(at 1197.61 1202.69 0)
+			(at 822.96 62.23 0)
 			(hide yes)
 			(show_name no)
@@
 		)
 		(property "Datasheet" ""
-			(at 1197.61 1202.69 0)
+			(at 822.96 62.23 0)
 			(hide yes)
 			(show_name no)
@@
 		)
 		(property "Description" "Power symbol creates a global label with name \"+5V\""
-			(at 1197.61 1202.69 0)
+			(at 822.96 62.23 0)
 			(hide yes)
 			(show_name no)
@@
 	(symbol
 		(lib_id "74xx:74HC74")
-		(at 1197.61 1210.31 0)
+		(at 822.96 69.85 0)
 		(unit 2)
 		(body_style 1)
@@
 		(fields_autoplaced yes)
 		(property "Reference" "U22"
-			(at 1199.7533 1200.15 0)
+			(at 825.1033 59.69 0)
 			(show_name no)
 			(do_not_autoplace no)
@@
 		)
 		(property "Value" "74HC74"
-			(at 1199.7533 1202.69 0)
+			(at 825.1033 62.23 0)
 			(show_name no)
 			(do_not_autoplace no)
@@
 		)
 		(property "Footprint" "Package_DIP:DIP-14_W10.16mm_LongPads"
-			(at 1197.61 1210.31 0)
+			(at 822.96 69.85 0)
 			(hide yes)
 			(show_name no)
@@
 		)
 		(property "Datasheet" "https://assets.nexperia.com/documents/data-sheet/74HC_HCT74.pdf"
-			(at 1197.61 1210.31 0)
+			(at 822.96 69.85 0)
 			(hide yes)
 			(show_name no)
@@
 		)
 		(property "Description" "Dual D Flip-flop, Set & Reset"
-			(at 1197.61 1210.31 0)
+			(at 822.96 69.85 0)
 			(hide yes)
 			(show_name no)
@@
 			)
 		)
-		(property "Footprint" ""
+		(property "Footprint" "Package_SO:TSSOP-14_4.4x5mm_P0.65mm"
 			(at 690.88 63.5 0)
 			(hide yes)
@@
 	(symbol
 		(lib_id "power:+5V")
-		(at 1200.15 1221.74 0)
+		(at 825.5 81.28 0)
 		(unit 1)
 		(body_style 1)
@@
 		(fields_autoplaced yes)
 		(property "Reference" "#PWR0558"
-			(at 1200.15 1225.55 0)
+			(at 825.5 85.09 0)
 			(hide yes)
 			(show_name no)
@@
 		)
 		(property "Value" "+5V"
-			(at 1200.15 1216.66 0)
+			(at 825.5 76.2 0)
 			(show_name no)
 			(do_not_autoplace no)
@@
 		)
 		(property "Footprint" ""
-			(at 1200.15 1221.74 0)
+			(at 825.5 81.28 0)
 			(hide yes)
 			(show_name no)
@@
 		)
 		(property "Datasheet" ""
-			(at 1200.15 1221.74 0)
+			(at 825.5 81.28 0)
 			(hide yes)
 			(show_name no)
@@
 		)
 		(property "Description" "Power symbol creates a global label with name \"+5V\""
-			(at 1200.15 1221.74 0)
+			(at 825.5 81.28 0)
 			(hide yes)
 			(show_name no)
@@
 			)
 		)
-		(property "Footprint" ""
+		(property "Footprint" "Package_SO:TSSOP-14_4.4x5mm_P0.65mm"
 			(at 751.84 45.72 0)
 			(hide yes)
@@
 			)
 		)
-		(property "Footprint" ""
+		(property "Footprint" "Package_SO:TSSOP-14_4.4x5mm_P0.65mm"
 			(at 750.57 82.55 0)
 			(hide yes)
@@
 	(symbol
 		(lib_id "power:GND")
-		(at 1187.45 1207.77 0)
+		(at 812.8 67.31 0)
 		(unit 1)
 		(body_style 1)
@@
 		(fields_autoplaced yes)
 		(property "Reference" "#PWR0556"
-			(at 1187.45 1214.12 0)
+			(at 812.8 73.66 0)
 			(hide yes)
 			(show_name no)
@@
 		)
 		(property "Value" "GND"
-			(at 1187.45 1212.85 0)
+			(at 812.8 72.39 0)
 			(show_name no)
 			(do_not_autoplace no)
@@
 		)
 		(property "Footprint" ""
-			(at 1187.45 1207.77 0)
+			(at 812.8 67.31 0)
 			(hide yes)
 			(show_name no)
@@
 		)
 		(property "Datasheet" ""
-			(at 1187.45 1207.77 0)
+			(at 812.8 67.31 0)
 			(hide yes)
 			(show_name no)
@@
 		)
 		(property "Description" "Power symbol creates a global label with name \"GND\" , ground"
-			(at 1187.45 1207.77 0)
+			(at 812.8 67.31 0)
 			(hide yes)
 			(show_name no)
@@
 			)
 		)
-		(property "Footprint" ""
+		(property "Footprint" "Package_SO:TSSOP-14_4.4x5mm_P0.65mm"
 			(at 731.52 45.72 0)
 			(hide yes)
@@
 			)
 		)
-		(property "Footprint" ""
+		(property "Footprint" "Package_SO:TSSOP-14_4.4x5mm_P0.65mm"
 			(at 731.52 100.33 0)
 			(hide yes)
@@
 			)
 		)
-		(property "Footprint" ""
+		(property "Footprint" "Package_SO:TSSOP-14_4.4x5mm_P0.65mm"
 			(at 730.25 64.77 0)
 			(hide yes)
@@
 			)
 		)
-		(property "Footprint" ""
+		(property "Footprint" "Package_SO:TSSOP-14_4.4x5mm_P0.65mm"
 			(at 711.2 81.28 0)
 			(hide yes)
@@
 			)
 		)
-		(property "Footprint" ""
+		(property "Footprint" "Package_SO:TSSOP-14_4.4x5mm_P0.65mm"
 			(at 711.2 63.5 0)
 			(hide yes)
@@
 			)
 		)
-		(property "Footprint" ""
+		(property "Footprint" "Package_SO:TSSOP-14_4.4x5mm_P0.65mm"
 			(at 730.25 82.55 0)
 			(hide yes)
@@
 			)
 		)
-		(property "Footprint" ""
+		(property "Footprint" "Package_SO:TSSOP-14_4.4x5mm_P0.65mm"
 			(at 668.02 81.28 0)
 			(hide yes)
@@
 			)
 		)
-		(property "Footprint" ""
+		(property "Footprint" "Package_SO:TSSOP-14_4.4x5mm_P0.65mm"
 			(at 692.15 99.06 0)
 			(hide yes)
@@
 			)
 		)
-		(property "Footprint" ""
+		(property "Footprint" "Package_SO:TSSOP-14_4.4x5mm_P0.65mm"
 			(at 690.88 81.28 0)
 			(hide yes)
@@
 			)
 		)
-		(property "Footprint" ""
+		(property "Footprint" "Package_SO:TSSOP-14_4.4x5mm_P0.65mm"
 			(at 711.2 45.72 0)
 			(hide yes)
@@
 			)
 		)
-		(property "Footprint" ""
+		(property "Footprint" "Package_SO:TSSOP-14_4.4x5mm_P0.65mm"
 			(at 646.43 63.5 0)
 			(hide yes)
@@
 			)
 		)
-		(property "Footprint" ""
+		(property "Footprint" "Package_SO:TSSOP-14_4.4x5mm_P0.65mm"
 			(at 646.43 45.72 0)
 			(hide yes)
@@
 			)
 		)
-		(property "Footprint" ""
+		(property "Footprint" "Package_SO:TSSOP-14_4.4x5mm_P0.65mm"
 			(at 690.88 45.72 0)
 			(hide yes)
@@
 			)
 		)
-		(property "Footprint" ""
+		(property "Footprint" "Package_SO:TSSOP-14_4.4x5mm_P0.65mm"
 			(at 668.02 63.5 0)
 			(hide yes)
